Commit message: fixing issues

File: drone_ws/src/drone_description/urdf/quadcopter.urdf (robot description, URDF)
Before this commit: robot quadcopter, 42 links, 41 joints
Links:
- removed link axis
- removed link mate_connector_1
- removed link mate_connector_10
- removed link mate_connector_11
- removed link mate_connector_2
- removed link mate_connector_3
- removed link mate_connector_4
- removed link mate_connector_5
- removed link mate_connector_6
- removed link mate_connector_7
- removed link mate_connector_8
- removed link mate_connector_9
- removed link part_1
- removed link part_1_1
- removed link part_1_10
- removed link part_1_11
- removed link part_1_12
- removed link part_1_13
- removed link part_1_14
- removed link part_1_15
- removed link part_1_16
- removed link part_1_17
- removed link part_1_18
- removed link part_1_19
- removed link part_1_2
- removed link part_1_20
- removed link part_1_21
- removed link part_1_22
- removed link part_1_23
- removed link part_1_24
- removed link part_1_25
- removed link part_1_26
- removed link part_1_27
- removed link part_1_28
- removed link part_1_3
- removed link part_1_4
- removed link part_1_5
- removed link part_1_6
- removed link part_1_7
- removed link part_1_8
- removed link part_1_9
- removed link root
- added link arm_link, mass 0.0122447; visual mesh filename=package://drone_description/meshes/Arm_link.stl scale=1 1 1
- added link arm_link_1, mass 0.0122447; visual mesh filename=package://drone_description/meshes/Arm_link.stl scale=1 1 1
- added link arm_link_2, mass 0.0122447; visual mesh filename=package://drone_description/meshes/Arm_link.stl scale=1 1 1
- added link arm_link_3, mass 0.0122447; visual mesh filename=package://drone_description/meshes/Arm_link.stl scale=1 1 1
- added link base_footprint
- added link base_link, mass 0.0173402; visual mesh filename=package://drone_description/meshes/base_link.stl scale=1 1 1
- added link board_link, mass 0.00355087; visual mesh filename=package://drone_description/meshes/Board_link.stl scale=1 1 1
- added link board_link_1, mass 0.00355087; visual mesh filename=package://drone_description/meshes/Board_link.stl scale=1 1 1
- added link imu_link, mass 0.002104; visual mesh filename=package://drone_description/meshes/imu_link.stl scale=1 1 1
- added link motor_link, mass 0.00882396; visual mesh filename=package://drone_description/meshes/Motor_link.stl scale=1 1 1
- added link motor_link_1, mass 0.00882396; visual mesh filename=package://drone_description/meshes/Motor_link.stl scale=1 1 1
- added link motor_link_2, mass 0.00882396; visual mesh filename=package://drone_description/meshes/Motor_link.stl scale=1 1 1
- added link motor_link_3, mass 0.00882396; visual mesh filename=package://drone_description/meshes/Motor_link.stl scale=1 1 1
- added link pillar_link, mass 0.000216885; visual mesh filename=package://drone_description/meshes/Pillar_link.stl scale=1 1 1
- added link pillar_link_1, mass 0.000216885; visual mesh filename=package://drone_description/meshes/Pillar_link.stl scale=1 1 1
- added link pillar_link_2, mass 0.000216885; visual mesh filename=package://drone_description/meshes/Pillar_link.stl scale=1 1 1
- added link pillar_link_3, mass 0.000216885; visual mesh filename=package://drone_description/meshes/Pillar_link.stl scale=1 1 1
- added link propeller_link, mass 0.00103601; visual mesh filename=package://drone_description/meshes/Propeller_link.stl scale=1 1 1
- added link propeller_link_1, mass 0.00103601; visual mesh filename=package://drone_description/meshes/Propeller_link.stl scale=1 1 1
- added link propeller_link_2, mass 0.00103601; visual mesh filename=package://drone_description/meshes/Propeller_link.stl scale=1 1 1
- added link propeller_link_3, mass 0.00103601; visual mesh filename=package://drone_description/meshes/Propeller_link.stl scale=1 1 1
- added link spacer_link, mass 0.000120637; visual mesh filename=package://drone_description/meshes/Spacer_link.stl scale=1 1 1
- added link spacer_link_1, mass 0.000120637; visual mesh filename=package://drone_description/meshes/Spacer_link.stl scale=1 1 1
- added link spacer_link_2, mass 0.000120637; visual mesh filename=package://drone_description/meshes/Spacer_link.stl scale=1 1 1
- added link spacer_link_3, mass 0.000120637; visual mesh filename=package://drone_description/meshes/Spacer_link.stl scale=1 1 1
- added link spinner_link, mass 0.00113254; visual mesh filename=package://drone_description/meshes/Spinner_link.stl scale=1 1 1
- added link spinner_link_1, mass 0.00113254; visual mesh filename=package://drone_description/meshes/Spinner_link.stl scale=1 1 1
- added link spinner_link_2, mass 0.00113254; visual mesh filename=package://drone_description/meshes/Spinner_link.stl scale=1 1 1
- added link spinner_link_3, mass 0.00113254; visual mesh filename=package://drone_description/meshes/Spinner_link.stl scale=1 1 1
- added link top_link, mass 0.0175978; visual mesh filename=package://drone_description/meshes/Top_link.stl scale=1 1 1
Joints:
- removed joint axis
- removed joint fastened_1
- removed joint fastened_11
- removed joint fastened_4
- removed joint fastened_5
- removed joint fastened_6
- removed joint fastened_7
- removed joint fastened_8
- removed joint fastened_9
- removed joint fastened_9_1
- removed joint fastened_9_2
- removed joint fastened_9_3
- removed joint hanging_node_to_root_joint
- removed joint mate_connector_1
- removed joint mate_connector_10
- removed joint mate_connector_11
- removed joint mate_connector_2
- removed joint mate_connector_3
- removed joint mate_connector_4
- removed joint mate_connector_5
- removed joint mate_connector_6
- removed joint mate_connector_7
- removed joint mate_connector_8
- removed joint mate_connector_9
- removed joint revolute_1
- removed joint revolute_1_1
- removed joint revolute_1_2
- removed joint revolute_1_3
- removed joint revolute_3
- removed joint revolute_5
- removed joint revolute_5_1
- removed joint revolute_5_2
- removed joint revolute_5_3
- removed joint revolute_6
- removed joint revolute_6_1
- removed joint revolute_6_2
- removed joint revolute_6_3
- removed joint revolute_7
- removed joint revolute_7_1
- removed joint revolute_7_2
- removed joint revolute_7_3
- added joint arms_top_1_joint: type continuous, parent top_link, child arm_link, origin xyz=0.0311127 -0.0226274 0.0041 rpy=-3.14159 -4.28599e-17 0.785398, axis -0 -0 1
- added joint base_board1_joint: type fixed, parent base_link, child board_link, origin xyz=0.0463627 0.00737742 -0.0005 rpy=2.11916e-17 -4.90352e-18 -4.996e-16, axis 0 0 -1
- added joint base_joint: type fixed, parent base_footprint, child base_link, origin xyz=0 0 0.008 rpy=0 0 0
- added joint base_top_joint: type fixed, parent base_link, child top_link, origin xyz=-0.0814963 0.0335523 0.0258382 rpy=-3.14159 2.13437e-16 -2.39915, axis 0 0 1
- added joint board2_imu_joint: type fixed, parent board_link_1, child imu_link, origin xyz=0.01525 0.01525 -0.00175 rpy=-3.14159 1.38667e-32 -3.14159, axis 0 0 -1
- added joint motor1_spinner1_joint: type continuous, parent motor_link_1, child spinner_link_3, origin xyz=2.77556e-17 1.38778e-17 0.0185 rpy=-7.64093e-18 3.26804e-18 0.0429589, axis -0 -0 -1
- added joint motor2_spinner2_joint: type continuous, parent motor_link_3, child spinner_link_1, origin xyz=0 3.46945e-18 0.0185 rpy=-8.55285e-50 2.46519e-32 -6.93889e-18, axis 0 0 -1
- added joint motor3_spinner3_joint: type continuous, parent motor_link, child spinner_link_2, origin xyz=0 2.77556e-17 0.0185 rpy=0 -0 2.902e-33, axis 0 0 -1
- added joint motor4_spinner4_joint: type continuous, parent motor_link_2, child spinner_link, origin xyz=0 0 0.0185 rpy=1.2326e-32 1.2326e-32 -6.93889e-18, axis 0 0 -1
- added joint rear_left_arm_base_1_joint: type fixed, parent base_link, child arm_link_3, origin xyz=0.00848528 0.0537401 -8.67362e-19 rpy=1.11911e-17 -1.72107e-17 1.94289e-16, axis 0 0 -1
- added joint rear_left_arm_motor4_joint: type continuous, parent arm_link_3, child motor_link_2, origin xyz=-0.0622254 0.0537401 0.0045 rpy=-6.38197e-33 1.54074e-32 -0.785398, axis 0 0 -1
- added joint rear_left_arm_pillar4_joint: type fixed, parent arm_link_3, child pillar_link, origin xyz=-0.0481437 0.0332945 -1.73472e-18 rpy=-3.14159 -1.54074e-32 2.35619, axis 0 0 -1
- added joint rear_left_board1_spacer_joint: type fixed, parent board_link, child spacer_link, origin xyz=-0.0305 0.0305 0.00175 rpy=2.46519e-32 1.38667e-32 -5.55112e-17, axis 0 0 -1
- added joint rear_right_arm_base_1_joint: type fixed, parent base_link, child arm_link_2, origin xyz=0.0537401 0.0537401 -1.30104e-18 rpy=1.24836e-16 1.19119e-17 -1.5708, axis 0 0 -1
- added joint rear_right_arm_motor3_joint: type continuous, parent arm_link_2, child motor_link, origin xyz=-0.0537401 0.0622254 0.0045 rpy=-4.11167e-32 3.14719e-32 0.785398, axis 0 0 -1
- added joint rear_right_arm_pillar3_joint: type fixed, parent arm_link_2, child pillar_link_1, origin xyz=-0.0396584 0.0417797 -2.38524e-18 rpy=-3.14159 -3.14719e-32 -2.35619, axis 0 0 -1
- added joint rear_right_board1_spacer_joint: type fixed, parent board_link, child spacer_link_3, origin xyz=-3.46945e-18 0.0305 0.00175 rpy=2.46519e-32 1.38667e-32 -5.55112e-17, axis 0 0 -1
- added joint spacers_board2_joint: type fixed, parent spacer_link_2, child board_link_1, origin xyz=0 0 0.006 rpy=3.14159 -3.08149e-33 -3.14159, axis 0 0 1
- added joint spinner1_propeller1_joint: type continuous, parent spinner_link_3, child propeller_link_2, origin xyz=0 0 0.0035 rpy=0 -0 0, axis 0 0 -1
- added joint spinner2_propeller2_joint: type continuous, parent spinner_link_1, child propeller_link_1, origin xyz=-6.93889e-18 0 0.0035 rpy=-8.55285e-50 2.46519e-32 -6.93889e-18, axis 0 0 -1
- added joint spinner3_propeller3_joint: type continuous, parent spinner_link_2, child propeller_link_3, origin xyz=0 2.77556e-17 0.0035 rpy=0 -0 2.902e-33, axis 0 0 -1
- added joint spinner4_propeller4_joint: type continuous, parent spinner_link, child propeller_link, origin xyz=0 0 0.0035 rpy=1.2326e-32 1.2326e-32 -6.93889e-18, axis 0 0 -1
- added joint top_left_arm_base_1_joint: type fixed, parent arm_link, child base_link, origin xyz=-1.38778e-17 -1.73472e-18 -0.02 rpy=-2.81271e-17 6.53168e-17 -2.35619, axis -0 -0 1
- added joint top_left_arm_motor1_joint: type continuous, parent arm_link, child motor_link_1, origin xyz=-0.006 0.082 -0.0155 rpy=2.09423e-16 2.59744e-16 3.14159, axis 0 0 -1
- added joint top_left_arm_pillar1_joint: type fixed, parent arm_link, child pillar_link_2, origin xyz=-0.0105 0.0575855 -0.02 rpy=-3.14159 1.2326e-32 6.93889e-18, axis 0 0 -1
- added joint top_left_board1_spacer_joint: type fixed, parent board_link, child spacer_link_1, origin xyz=-0.0305 0 0.00175 rpy=2.46519e-32 1.38667e-32 -5.55112e-17, axis 0 0 -1
- added joint top_right_arm_base_1_joint: type fixed, parent base_link, child arm_link_1, origin xyz=0.0622254 2.08167e-17 0 rpy=4.15504e-17 2.70178e-17 4.996e-16, axis 0 0 -1
- added joint top_right_arm_motor2_joint: type continuous, parent arm_link_1, child motor_link_3, origin xyz=0.0537401 -0.0622254 0.0045 rpy=-1.02112e-32 2.46519e-32 -0.785398, axis 0 0 -1
- added joint top_right_arm_pillar2_joint: type fixed, parent arm_link_1, child pillar_link_3, origin xyz=0.0396584 -0.0417797 -2.1684e-19 rpy=-3.14159 -2.46519e-32 2.35619, axis 0 0 -1
- added joint top_right_board1_spacer_joint: type fixed, parent board_link, child spacer_link_2, origin xyz=0 0 0.00175 rpy=2.46519e-32 1.38667e-32 -5.55112e-17, axis 0 0 -1
