Commit message: adding launch, world and rivz files

File: drone_ws/src/drone_description/urdf/quadcopter.urdf.xacro (robot description, xacro)
@@ -1,3 +1,6 @@
-<robot name="quadcopter">
+<?xml version="1.0"?>
+<robot xmlns:xacro="http://www.ros.org/wiki/xacro" name="quadcopter">
+    <xacro:arg name="is_ignition" default="true"/>
+    <xacro:include filename="$(find drone_description)/urdf/quadcopter_gazebo.xacro"/>
     <link name="base_footprint"/>
     <link name="arm_link">
@@ -491,5 +494,5 @@
         <origin xyz="-0.0814963 0.0335523 0.0258382" rpy="-3.14159 2.13437e-16 -2.39915" />
         <axis xyz="0 0 1" />
-        <parent link="base_link" />
+        <parent link="base_footprint" />
         <child link="top_link" />
     </joint>
@@ -524,5 +527,5 @@
         <child link="arm_link_3" />
     </joint>
-    <joint name="rear_left_arm_motor4_joint" type="continuous">
+    <joint name="rear_left_arm_motor4_joint" type="fixed">
         <origin xyz="-0.0622254 0.0537401 0.0045" rpy="-6.38197e-33 1.54074e-32 -0.785398" />
         <axis xyz="0 0 -1" />
@@ -548,5 +551,5 @@
         <child link="arm_link_2" />
     </joint>
-    <joint name="rear_right_arm_motor3_joint" type="continuous">
+    <joint name="rear_right_arm_motor3_joint" type="fixed">
         <origin xyz="-0.0537401 0.0622254 0.0045" rpy="-4.11167e-32 3.14719e-32 0.785398" />
         <axis xyz="0 0 -1" />
@@ -572,5 +575,5 @@
         <child link="board_link_1" />
     </joint>
-    <joint name="spinner1_propeller1_joint" type="continuous">
+    <joint name="spinner1_propeller1_joint" type="fixed">
         <origin xyz="0 0 0.0035" rpy="0 -0 0" />
         <axis xyz="0 0 -1" />
@@ -578,5 +581,5 @@
         <child link="propeller_link_2" />
     </joint>
-    <joint name="spinner2_propeller2_joint" type="continuous">
+    <joint name="spinner2_propeller2_joint" type="fixed">
         <origin xyz="-6.93889e-18 0 0.0035" rpy="-8.55285e-50 2.46519e-32 -6.93889e-18" />
         <axis xyz="0 0 -1" />
@@ -584,5 +587,5 @@
         <child link="propeller_link_1" />
     </joint>
-    <joint name="spinner3_propeller3_joint" type="continuous">
+    <joint name="spinner3_propeller3_joint" type="fixed">
         <origin xyz="0 2.77556e-17 0.0035" rpy="0 -0 2.902e-33" />
         <axis xyz="0 0 -1" />
@@ -590,5 +593,5 @@
         <child link="propeller_link_3" />
     </joint>
-    <joint name="spinner4_propeller4_joint" type="continuous">
+    <joint name="spinner4_propeller4_joint" type="fixed">
         <origin xyz="0 0 0.0035" rpy="1.2326e-32 1.2326e-32 -6.93889e-18" />
         <axis xyz="0 0 -1" />
@@ -602,5 +605,5 @@
         <child link="base_link" />
     </joint>
-    <joint name="top_left_arm_motor1_joint" type="continuous">
+    <joint name="top_left_arm_motor1_joint" type="fixed">
         <origin xyz="-0.006 0.082 -0.0155" rpy="2.09423e-16 2.59744e-16 3.14159" />
         <axis xyz="0 0 -1" />
@@ -626,5 +629,5 @@
         <child link="arm_link_1" />
     </joint>
-    <joint name="top_right_arm_motor2_joint" type="continuous">
+    <joint name="top_right_arm_motor2_joint" type="fixed">
         <origin xyz="0.0537401 -0.0622254 0.0045" rpy="-1.02112e-32 2.46519e-32 -0.785398" />
         <axis xyz="0 0 -1" />

Commit message: adding yaml parameters for the melllinger controller

File: drone_ws/src/drone_description/urdf/quadcopter.urdf.xacro (robot description, xacro)
@@ -1,8 +1,6 @@
 <?xml version="1.0"?>
 <robot xmlns:xacro="http://www.ros.org/wiki/xacro" name="quadcopter">
-    <!--
     <xacro:arg name="is_ignition" default="true"/>
     <xacro:include filename="$(find drone_description)/urdf/quadcopter_gazebo.xacro"/>
-    -->
     <link name="base_footprint"/>
     <link name="arm_link">
@@ -21,4 +19,10 @@
             </material>
         </visual>
+        <collision>
+            <origin xyz="-0.015 -0.004 -0.02" rpy="0 -0 0" />
+            <geometry>
+                <mesh filename="package://drone_description/meshes/Arm_link.stl"/>
+            </geometry>
+        </collision>
     </link>
     <link name="arm_link_1">
@@ -37,4 +41,10 @@
             </material>
         </visual>
+        <collision>
+            <origin xyz="-0.000707107 0.00494975 0" rpy="0 -0 -2.35619" />
+            <geometry>
+                <mesh filename="package://drone_description/meshes/Arm_link.stl"/>
+            </geometry>
+        </collision>
     </link>
     <link name="arm_link_2">
@@ -53,4 +63,10 @@
             </material>
         </visual>
+        <collision>
+            <origin xyz="0.000707107 -0.00494975 0" rpy="0 -0 0.785398" />
+            <geometry>
+                <mesh filename="package://drone_description/meshes/Arm_link.stl"/>
+            </geometry>
+        </collision>
     </link>
     <link name="arm_link_3">
@@ -69,4 +85,10 @@
             </material>
         </visual>
+        <collision>
+            <origin xyz="-0.00777817 -0.013435 0" rpy="0 -0 0.785398" />
+            <geometry>
+                <mesh filename="package://drone_description/meshes/Arm_link.stl"/>
+            </geometry>
+        </collision>
     </link>
     <link name="base_link">
@@ -85,4 +107,10 @@
             </material>
         </visual>
+        <collision>
+            <origin xyz="0.0311127 0.0226274 -0.004" rpy="0 -0 0" />
+            <geometry>
+                <mesh filename="package://drone_description/meshes/base_link.stl"/>
+            </geometry>
+        </collision>
     </link>
     <link name="board_link">
@@ -101,4 +129,10 @@
             </material>
         </visual>
+        <collision>
+            <origin xyz="-0.01525 0.01525 0" rpy="0 -0 0" />
+            <geometry>
+                <mesh filename="package://drone_description/meshes/Board_link.stl"/>
+            </geometry>
+        </collision>
     </link>
     <link name="board_link_1">
@@ -117,4 +151,10 @@
             </material>
         </visual>
+        <collision>
+            <origin xyz="0.01525 0.01525 -0.00175" rpy="0 -0 0" />
+            <geometry>
+                <mesh filename="package://drone_description/meshes/Board_link.stl"/>
+            </geometry>
+        </collision>
     </link>
     <link name="imu_link">
@@ -133,4 +173,10 @@
             </material>
         </visual>
+        <collision>
+            <origin xyz="1.4456e-19 3.97541e-19 0" rpy="0 -0 0" />
+            <geometry>
+                <mesh filename="package://drone_description/meshes/imu_link.stl"/>
+            </geometry>
+        </collision>
     </link>
     <link name="motor_link">
@@ -149,4 +195,10 @@
             </material>
         </visual>
+        <collision>
+            <origin xyz="0 0 0" rpy="0 -0 0" />
+            <geometry>
+                <mesh filename="package://drone_description/meshes/Motor_link.stl"/>
+            </geometry>
+        </collision>
     </link>
     <link name="motor_link_1">
@@ -165,4 +217,10 @@
             </material>
         </visual>
+        <collision>
+            <origin xyz="0 0 0" rpy="0 -0 0.0429589" />
+            <geometry>
+                <mesh filename="package://drone_description/meshes/Motor_link.stl"/>
+            </geometry>
+        </collision>
     </link>
     <link name="motor_link_2">
@@ -181,4 +239,10 @@
             </material>
         </visual>
+        <collision>
+            <origin xyz="0 0 0" rpy="0 -0 0" />
+            <geometry>
+                <mesh filename="package://drone_description/meshes/Motor_link.stl"/>
+            </geometry>
+        </collision>
     </link>
     <link name="motor_link_3">
@@ -197,4 +261,10 @@
             </material>
         </visual>
+        <collision>
+            <origin xyz="0 0 0" rpy="0 -0 0" />
+            <geometry>
+                <mesh filename="package://drone_description/meshes/Motor_link.stl"/>
+            </geometry>
+        </collision>
     </link>
     <link name="pillar_link">
@@ -213,4 +283,10 @@
             </material>
         </visual>
+        <collision>
+            <origin xyz="0 -7.65404e-20 -0.0039" rpy="0 -0 0" />
+            <geometry>
+                <mesh filename="package://drone_description/meshes/Pillar_link.stl"/>
+            </geometry>
+        </collision>
     </link>
     <link name="pillar_link_1">
@@ -229,4 +305,10 @@
             </material>
         </visual>
+        <collision>
+            <origin xyz="0 -7.65404e-20 -0.0039" rpy="0 -0 0" />
+            <geometry>
+                <mesh filename="package://drone_description/meshes/Pillar_link.stl"/>
+            </geometry>
+        </collision>
     </link>
     <link name="pillar_link_2">
@@ -245,4 +327,10 @@
             </material>
         </visual>
+        <collision>
+            <origin xyz="0 -7.65404e-20 -0.0039" rpy="0 -0 0" />
+            <geometry>
+                <mesh filename="package://drone_description/meshes/Pillar_link.stl"/>
+            </geometry>
+        </collision>
     </link>
     <link name="pillar_link_3">
@@ -261,4 +349,10 @@
             </material>
         </visual>
+        <collision>
+            <origin xyz="0 -7.65404e-20 -0.0039" rpy="0 -0 0" />
+            <geometry>
+                <mesh filename="package://drone_description/meshes/Pillar_link.stl"/>
+            </geometry>
+        </collision>
     </link>
     <link name="propeller_link">
@@ -341,4 +435,10 @@
             </material>
         </visual>
+        <collision>
+            <origin xyz="0 -9.18485e-20 0" rpy="0 -0 0" />
+            <geometry>
+                <mesh filename="package://drone_description/meshes/Spacer_link.stl"/>
+            </geometry>
+        </collision>
     </link>
     <link name="spacer_link_1">
@@ -357,4 +457,10 @@
             </material>
         </visual>
+        <collision>
+            <origin xyz="0 -9.18485e-20 0" rpy="0 -0 0" />
+            <geometry>
+                <mesh filename="package://drone_description/meshes/Spacer_link.stl"/>
+            </geometry>
+        </collision>
     </link>
     <link name="spacer_link_2">
@@ -373,4 +479,10 @@
             </material>
         </visual>
+        <collision>
+            <origin xyz="0 -9.18485e-20 0" rpy="0 -0 0" />
+            <geometry>
+                <mesh filename="package://drone_description/meshes/Spacer_link.stl"/>
+            </geometry>
+        </collision>
     </link>
     <link name="spacer_link_3">
@@ -389,4 +501,10 @@
             </material>
         </visual>
+        <collision>
+            <origin xyz="0 -9.18485e-20 0" rpy="0 -0 0" />
+            <geometry>
+                <mesh filename="package://drone_description/meshes/Spacer_link.stl" scale="1 1 1" />
+            </geometry>
+        </collision>
     </link>
     <link name="spinner_link">
@@ -469,4 +587,10 @@
             </material>
         </visual>
+        <collision>
+            <origin xyz="0 0 0" rpy="0 -0 0" />
+            <geometry>
+                <mesh filename="package://drone_description/meshes/Top_link.stl"/>
+            </geometry>
+        </collision>
     </link>
     <joint name="base_joint" type="fixed">

File: drone_ws/src/drone_description/urdf/quadcopter_gazebo.xacro (robot description, xacro)
@@ -4,5 +4,5 @@
         <xacro:if value="$(arg is_ignition)">
             <plugin filename="ign_ros2_control-system" name="ign_ros2_control::IgnitionROS2ControlPlugin">
-                <parameters>$(find bumperbot_controller)/config/bumperbot_controllers.yaml</parameters>
+                <parameters>$(find drone_controllers)/config/mellinger_controller.yaml</parameters>
             </plugin>
             <plugin filename="ignition-gazebo-imu-system" name="ignition::gazebo::systems::Imu">
@@ -11,9 +11,41 @@
         <xacro:unless value="$(arg is_ignition)">
             <plugin filename="gz_ros2_control-system" name="gz_ros2_control::GazeboSimROS2ControlPlugin">
-                <parameters>$(find bumperbot_controller)/config/bumperbot_controllers.yaml</parameters>
+                <parameters>$(find drone_controllers)/config/mellinger_controller.yaml</parameters>
             </plugin>
             <plugin filename="gz-sim-imu-system" name="gz::sim::systems::Imu">
             </plugin>
         </xacro:unless>
+    </gazebo>
+    <gazebo reference="pillar_link">
+        <mu1>0.8</mu1>
+        <mu2>0.8</mu2>
+        <kp>100000</kp>
+        <kd>10</kd>
+        <minDepth>0.001</minDepth>
+        <maxVel>0.1</maxVel>
+    </gazebo>
+    <gazebo reference="pillar_link_1">
+        <mu1>0.8</mu1>
+        <mu2>0.8</mu2>
+        <kp>100000</kp>
+        <kd>10</kd>
+        <minDepth>0.001</minDepth>
+        <maxVel>0.1</maxVel>
+    </gazebo>
+    <gazebo reference="pillar_link_2">
+        <mu1>0.8</mu1>
+        <mu2>0.8</mu2>
+        <kp>100000</kp>
+        <kd>10</kd>
+        <minDepth>0.001</minDepth>
+        <maxVel>0.1</maxVel>
+    </gazebo>
+    <gazebo reference="pillar_link_3">
+        <mu1>0.8</mu1>
+        <mu2>0.8</mu2>
+        <kp>100000</kp>
+        <kd>10</kd>
+        <minDepth>0.001</minDepth>
+        <maxVel>0.1</maxVel>
     </gazebo>
     <gazebo reference="imu_link">

Commit message: removing some bumperbot packages

File: drone_ws/src/drone_description/urdf/quadcopter.urdf.xacro (robot description, xacro)
@@ -729,6 +729,6 @@
         <origin xyz="-1.38778e-17 -1.73472e-18 -0.02" rpy="-2.81271e-17 6.53168e-17 -2.35619" />
         <axis xyz="-0 -0 1" />
-        <parent link="arm_link" />
-        <child link="base_link" />
+        <parent link="base_link" />
+        <child link="arm_link" />
     </joint>
     <joint name="top_left_arm_motor1_joint" type="fixed">

Commit message: .

File: drone_ws/src/drone_description/urdf/quadcopter.urdf.xacro (robot description, xacro)
@@ -1,8 +1,7 @@
-<?xml version="1.0"?>
-<robot xmlns:xacro="http://www.ros.org/wiki/xacro" name="quadcopter">
+<robot name="quadcopter" xmlns:xacro="http://www.ros.org/wiki/xacro">
     <xacro:arg name="is_ignition" default="true"/>
     <xacro:include filename="$(find drone_description)/urdf/quadcopter_gazebo.xacro"/>
     <xacro:include filename="$(find drone_description)/urdf/quadcopter_ros2_control.xacro"/>
-    <link name="base_footprint"/>
+    <link name="root" />
     <link name="arm_link">
         <inertial>
@@ -20,10 +19,4 @@
             </material>
         </visual>
-        <collision>
-            <origin xyz="-0.015 -0.004 -0.02" rpy="0 -0 0" />
-            <geometry>
-                <mesh filename="package://drone_description/meshes/Arm_link.stl"/>
-            </geometry>
-        </collision>
     </link>
     <link name="arm_link_1">
@@ -42,10 +35,4 @@
             </material>
         </visual>
-        <collision>
-            <origin xyz="-0.000707107 0.00494975 0" rpy="0 -0 -2.35619" />
-            <geometry>
-                <mesh filename="package://drone_description/meshes/Arm_link.stl"/>
-            </geometry>
-        </collision>
     </link>
     <link name="arm_link_2">
@@ -64,10 +51,4 @@
             </material>
         </visual>
-        <collision>
-            <origin xyz="0.000707107 -0.00494975 0" rpy="0 -0 0.785398" />
-            <geometry>
-                <mesh filename="package://drone_description/meshes/Arm_link.stl"/>
-            </geometry>
-        </collision>
     </link>
     <link name="arm_link_3">
@@ -86,10 +67,4 @@
             </material>
         </visual>
-        <collision>
-            <origin xyz="-0.00777817 -0.013435 0" rpy="0 -0 0.785398" />
-            <geometry>
-                <mesh filename="package://drone_description/meshes/Arm_link.stl"/>
-            </geometry>
-        </collision>
     </link>
     <link name="base_link">
@@ -108,10 +83,4 @@
             </material>
         </visual>
-        <collision>
-            <origin xyz="0.0311127 0.0226274 -0.004" rpy="0 -0 0" />
-            <geometry>
-                <mesh filename="package://drone_description/meshes/base_link.stl"/>
-            </geometry>
-        </collision>
     </link>
     <link name="board_link">
@@ -130,10 +99,4 @@
             </material>
         </visual>
-        <collision>
-            <origin xyz="-0.01525 0.01525 0" rpy="0 -0 0" />
-            <geometry>
-                <mesh filename="package://drone_description/meshes/Board_link.stl"/>
-            </geometry>
-        </collision>
     </link>
     <link name="board_link_1">
@@ -152,10 +115,4 @@
             </material>
         </visual>
-        <collision>
-            <origin xyz="0.01525 0.01525 -0.00175" rpy="0 -0 0" />
-            <geometry>
-                <mesh filename="package://drone_description/meshes/Board_link.stl"/>
-            </geometry>
-        </collision>
     </link>
     <link name="imu_link">
@@ -174,10 +131,4 @@
             </material>
         </visual>
-        <collision>
-            <origin xyz="1.4456e-19 3.97541e-19 0" rpy="0 -0 0" />
-            <geometry>
-                <mesh filename="package://drone_description/meshes/imu_link.stl"/>
-            </geometry>
-        </collision>
     </link>
     <link name="motor_link">
@@ -196,10 +147,4 @@
             </material>
         </visual>
-        <collision>
-            <origin xyz="0 0 0" rpy="0 -0 0" />
-            <geometry>
-                <mesh filename="package://drone_description/meshes/Motor_link.stl"/>
-            </geometry>
-        </collision>
     </link>
     <link name="motor_link_1">
@@ -218,10 +163,4 @@
             </material>
         </visual>
-        <collision>
-            <origin xyz="0 0 0" rpy="0 -0 0.0429589" />
-            <geometry>
-                <mesh filename="package://drone_description/meshes/Motor_link.stl"/>
-            </geometry>
-        </collision>
     </link>
     <link name="motor_link_2">
@@ -240,10 +179,4 @@
             </material>
         </visual>
-        <collision>
-            <origin xyz="0 0 0" rpy="0 -0 0" />
-            <geometry>
-                <mesh filename="package://drone_description/meshes/Motor_link.stl"/>
-            </geometry>
-        </collision>
     </link>
     <link name="motor_link_3">
@@ -262,10 +195,4 @@
             </material>
         </visual>
-        <collision>
-            <origin xyz="0 0 0" rpy="0 -0 0" />
-            <geometry>
-                <mesh filename="package://drone_description/meshes/Motor_link.stl"/>
-            </geometry>
-        </collision>
     </link>
     <link name="pillar_link">
@@ -284,10 +211,4 @@
             </material>
         </visual>
-        <collision>
-            <origin xyz="0 -7.65404e-20 -0.0039" rpy="0 -0 0" />
-            <geometry>
-                <mesh filename="package://drone_description/meshes/Pillar_link.stl"/>
-            </geometry>
-        </collision>
     </link>
     <link name="pillar_link_1">
@@ -306,10 +227,4 @@
             </material>
         </visual>
-        <collision>
-            <origin xyz="0 -7.65404e-20 -0.0039" rpy="0 -0 0" />
-            <geometry>
-                <mesh filename="package://drone_description/meshes/Pillar_link.stl"/>
-            </geometry>
-        </collision>
     </link>
     <link name="pillar_link_2">
@@ -328,10 +243,4 @@
             </material>
         </visual>
-        <collision>
-            <origin xyz="0 -7.65404e-20 -0.0039" rpy="0 -0 0" />
-            <geometry>
-                <mesh filename="package://drone_description/meshes/Pillar_link.stl"/>
-            </geometry>
-        </collision>
     </link>
     <link name="pillar_link_3">
@@ -350,10 +259,4 @@
             </material>
         </visual>
-        <collision>
-            <origin xyz="0 -7.65404e-20 -0.0039" rpy="0 -0 0" />
-            <geometry>
-                <mesh filename="package://drone_description/meshes/Pillar_link.stl"/>
-            </geometry>
-        </collision>
     </link>
     <link name="propeller_link">
@@ -436,10 +339,4 @@
             </material>
         </visual>
-        <collision>
-            <origin xyz="0 -9.18485e-20 0" rpy="0 -0 0" />
-            <geometry>
-                <mesh filename="package://drone_description/meshes/Spacer_link.stl"/>
-            </geometry>
-        </collision>
     </link>
     <link name="spacer_link_1">
@@ -458,10 +355,4 @@
             </material>
         </visual>
-        <collision>
-            <origin xyz="0 -9.18485e-20 0" rpy="0 -0 0" />
-            <geometry>
-                <mesh filename="package://drone_description/meshes/Spacer_link.stl"/>
-            </geometry>
-        </collision>
     </link>
     <link name="spacer_link_2">
@@ -480,10 +371,4 @@
             </material>
         </visual>
-        <collision>
-            <origin xyz="0 -9.18485e-20 0" rpy="0 -0 0" />
-            <geometry>
-                <mesh filename="package://drone_description/meshes/Spacer_link.stl"/>
-            </geometry>
-        </collision>
     </link>
     <link name="spacer_link_3">
@@ -502,10 +387,4 @@
             </material>
         </visual>
-        <collision>
-            <origin xyz="0 -9.18485e-20 0" rpy="0 -0 0" />
-            <geometry>
-                <mesh filename="package://drone_description/meshes/Spacer_link.stl" scale="1 1 1" />
-            </geometry>
-        </collision>
     </link>
     <link name="spinner_link">
@@ -588,17 +467,6 @@
             </material>
         </visual>
-        <collision>
-            <origin xyz="0 0 0" rpy="0 -0 0" />
-            <geometry>
-                <mesh filename="package://drone_description/meshes/Top_link.stl"/>
-            </geometry>
-        </collision>
-    </link>
-    <joint name="base_joint" type="fixed">
-        <parent link="base_footprint" />
-        <child link="base_link" />
-        <origin xyz="0 0 0.008" rpy="0 0 0" />
-    </joint>
-    <joint name="arms_top_1_joint" type="continuous">
+    </link>
+    <joint name="arms_top_1_joint" type="fixed">
         <origin xyz="0.0311127 -0.0226274 0.0041" rpy="-3.14159 -4.28599e-17 0.785398" />
         <axis xyz="-0 -0 1" />
@@ -618,8 +486,8 @@
         <child link="imu_link" />
     </joint>
-    <joint name="base_top_joint" type="fixed">
+    <joint name="hanging_node_to_root_joint" type="fixed">
         <origin xyz="-0.0814963 0.0335523 0.0258382" rpy="-3.14159 2.13437e-16 -2.39915" />
         <axis xyz="0 0 1" />
-        <parent link="base_footprint" />
+        <parent link="root" />
         <child link="top_link" />
     </joint>
@@ -729,6 +597,6 @@
         <origin xyz="-1.38778e-17 -1.73472e-18 -0.02" rpy="-2.81271e-17 6.53168e-17 -2.35619" />
         <axis xyz="-0 -0 1" />
-        <parent link="base_link" />
-        <child link="arm_link" />
+        <parent link="arm_link" />
+        <child link="base_link" />
     </joint>
     <joint name="top_left_arm_motor1_joint" type="fixed">
