Commit message: adding controller.launch.py

File: drone_ws/src/drone_description/urdf/quadcopter.urdf.xacro (robot description, xacro)
@@ -1,3 +1,3 @@
-<robot name="quadcopter" xmlns:xacro="http://www.ros.org/wiki/xacro">
+<robot name="quadcopter" xmlns:xacro="https://www.ros.org/wiki/xacro">
     <xacro:arg name="is_ignition" default="true"/>
     <xacro:include filename="$(find drone_description)/urdf/quadcopter_gazebo.xacro"/>
@@ -7,9 +7,9 @@
         <inertial>
             <mass value="0.0122447" />
-            <origin xyz="-0.00887441 0.0315104 -0.013797" rpy="0 -0 0" />
-            <inertia ixx="1.01513e-05" ixy="2.79072e-07" ixz="-3.24984e-08" iyy="5.30709e-07" iyz="8.08127e-07" izz="1.00597e-05" />
-        </inertial>
-        <visual>
-            <origin xyz="-0.015 -0.004 -0.02" rpy="0 -0 0" />
+            <origin xyz="-0.0285564 0.0160061 0.00620303" rpy="0 -0 0.785398" />
+            <inertia ixx="5.06194e-06" ixy="4.8103e-06" ixz="-5.94412e-07" iyy="5.62008e-06" iyz="5.48452e-07" izz="1.00597e-05" />
+        </inertial>
+        <visual>
+            <origin xyz="-0.00777817 -0.013435 0" rpy="0 -0 0.785398" />
             <geometry>
                 <mesh filename="package://drone_description/meshes/Arm_link.stl" scale="1 1 1" />
@@ -19,4 +19,10 @@
             </material>
         </visual>
+        <collision>
+            <origin xyz="-0.00777817 -0.013435 0" rpy="0 -0 0.785398" />
+            <geometry>
+                <mesh filename="package://drone_description/meshes/Arm_link.stl" scale="1 1 1" />
+            </geometry>
+        </collision>
     </link>
     <link name="arm_link_1">
@@ -35,4 +41,10 @@
             </material>
         </visual>
+        <collision>
+            <origin xyz="-0.000707107 0.00494975 0" rpy="0 -0 -2.35619" />
+            <geometry>
+                <mesh filename="package://drone_description/meshes/Arm_link.stl" scale="1 1 1" />
+            </geometry>
+        </collision>
     </link>
     <link name="arm_link_2">
@@ -51,4 +63,10 @@
             </material>
         </visual>
+        <collision>
+            <origin xyz="0.000707107 -0.00494975 0" rpy="0 -0 0.785398" />
+            <geometry>
+                <mesh filename="package://drone_description/meshes/Arm_link.stl" scale="1 1 1" />
+            </geometry>
+        </collision>
     </link>
     <link name="arm_link_3">
@@ -67,13 +85,19 @@
             </material>
         </visual>
+        <collision>
+            <origin xyz="-0.00777817 -0.013435 0" rpy="0 -0 0.785398" />
+            <geometry>
+                <mesh filename="package://drone_description/meshes/Arm_link.stl" scale="1 1 1" />
+            </geometry>
+        </collision>
     </link>
     <link name="base_link">
         <inertial>
             <mass value="0.0173402" />
-            <origin xyz="0.0311127 0.0226274 -0.00241704" rpy="0 -0 0" />
+            <origin xyz="1.23741e-17 -4.31023e-18 0.00558296" rpy="0 -0 0" />
             <inertia ixx="8.0893e-06" ixy="0" ixz="0" iyy="8.0893e-06" iyz="0" izz="1.61357e-05" />
         </inertial>
         <visual>
-            <origin xyz="0.0311127 0.0226274 -0.004" rpy="0 -0 0" />
+            <origin xyz="4.91335e-18 -1.08551e-18 0.004" rpy="0 -0 0" />
             <geometry>
                 <mesh filename="package://drone_description/meshes/base_link.stl" scale="1 1 1" />
@@ -83,4 +107,10 @@
             </material>
         </visual>
+        <collision>
+            <origin xyz="4.91335e-18 -1.08551e-18 0.004" rpy="0 -0 0" />
+            <geometry>
+                <mesh filename="package://drone_description/meshes/base_link.stl" scale="1 1 1" />
+            </geometry>
+        </collision>
     </link>
     <link name="board_link">
@@ -99,4 +129,10 @@
             </material>
         </visual>
+        <collision>
+            <origin xyz="-0.01525 0.01525 0" rpy="0 -0 0" />
+            <geometry>
+                <mesh filename="package://drone_description/meshes/Board_link.stl" scale="1 1 1" />
+            </geometry>
+        </collision>
     </link>
     <link name="board_link_1">
@@ -115,4 +151,10 @@
             </material>
         </visual>
+        <collision>
+            <origin xyz="0.01525 0.01525 -0.00175" rpy="0 -0 0" />
+            <geometry>
+                <mesh filename="package://drone_description/meshes/Board_link.stl" scale="1 1 1" />
+            </geometry>
+        </collision>
     </link>
     <link name="imu_link">
@@ -131,13 +173,19 @@
             </material>
         </visual>
+        <collision>
+            <origin xyz="1.4456e-19 3.97541e-19 0" rpy="0 -0 0" />
+            <geometry>
+                <mesh filename="package://drone_description/meshes/imu_link.stl" scale="1 1 1" />
+            </geometry>
+        </collision>
     </link>
     <link name="motor_link">
         <inertial>
             <mass value="0.00882396" />
-            <origin xyz="2.40215e-19 -1.21395e-18 0.00731802" rpy="0 -0 0" />
-            <inertia ixx="4.49229e-07" ixy="0" ixz="0" iyy="4.48384e-07" iyz="0" izz="5.69462e-07" />
-        </inertial>
-        <visual>
-            <origin xyz="0 0 0" rpy="0 -0 0" />
+            <origin xyz="9.97732e-19 -7.32058e-19 0.00731802" rpy="0 -0 0.742439" />
+            <inertia ixx="4.48843e-07" ixy="4.20673e-10" ixz="0" iyy="4.4877e-07" iyz="0" izz="5.69462e-07" />
+        </inertial>
+        <visual>
+            <origin xyz="0 0 0" rpy="0 -0 0.742439" />
             <geometry>
                 <mesh filename="package://drone_description/meshes/Motor_link.stl" scale="1 1 1" />
@@ -147,13 +195,19 @@
             </material>
         </visual>
+        <collision>
+            <origin xyz="0 0 0" rpy="0 -0 0.742439" />
+            <geometry>
+                <mesh filename="package://drone_description/meshes/Motor_link.stl" scale="1 1 1" />
+            </geometry>
+        </collision>
     </link>
     <link name="motor_link_1">
         <inertial>
             <mass value="0.00882396" />
-            <origin xyz="2.92128e-19 -1.20251e-18 0.00731802" rpy="0 -0 0.0429589" />
-            <inertia ixx="4.49227e-07" ixy="3.62325e-11" ixz="0" iyy="4.48386e-07" iyz="0" izz="5.69462e-07" />
-        </inertial>
-        <visual>
-            <origin xyz="0 0 0" rpy="0 -0 0.0429589" />
+            <origin xyz="1.02825e-18 -6.88534e-19 0.00731802" rpy="0 -0 0.785398" />
+            <inertia ixx="4.48807e-07" ixy="4.2223e-10" ixz="0" iyy="4.48807e-07" iyz="0" izz="5.69462e-07" />
+        </inertial>
+        <visual>
+            <origin xyz="0 0 0" rpy="0 -0 0.785398" />
             <geometry>
                 <mesh filename="package://drone_description/meshes/Motor_link.stl" scale="1 1 1" />
@@ -163,13 +217,19 @@
             </material>
         </visual>
+        <collision>
+            <origin xyz="0 0 0" rpy="0 -0 0.785398" />
+            <geometry>
+                <mesh filename="package://drone_description/meshes/Motor_link.stl" scale="1 1 1" />
+            </geometry>
+        </collision>
     </link>
     <link name="motor_link_2">
         <inertial>
             <mass value="0.00882396" />
-            <origin xyz="2.40215e-19 -1.21395e-18 0.00731802" rpy="0 -0 0" />
-            <inertia ixx="4.49229e-07" ixy="0" ixz="0" iyy="4.48384e-07" iyz="0" izz="5.69462e-07" />
-        </inertial>
-        <visual>
-            <origin xyz="0 0 0" rpy="0 -0 0" />
+            <origin xyz="9.97732e-19 -7.32058e-19 0.00731802" rpy="0 -0 0.742439" />
+            <inertia ixx="4.48843e-07" ixy="4.20673e-10" ixz="0" iyy="4.4877e-07" iyz="0" izz="5.69462e-07" />
+        </inertial>
+        <visual>
+            <origin xyz="0 0 0" rpy="0 -0 0.742439" />
             <geometry>
                 <mesh filename="package://drone_description/meshes/Motor_link.stl" scale="1 1 1" />
@@ -179,13 +239,19 @@
             </material>
         </visual>
+        <collision>
+            <origin xyz="0 0 0" rpy="0 -0 0.742439" />
+            <geometry>
+                <mesh filename="package://drone_description/meshes/Motor_link.stl" scale="1 1 1" />
+            </geometry>
+        </collision>
     </link>
     <link name="motor_link_3">
         <inertial>
             <mass value="0.00882396" />
-            <origin xyz="2.40215e-19 -1.21395e-18 0.00731802" rpy="0 -0 0" />
-            <inertia ixx="4.49229e-07" ixy="0" ixz="0" iyy="4.48384e-07" iyz="0" izz="5.69462e-07" />
-        </inertial>
-        <visual>
-            <origin xyz="0 0 0" rpy="0 -0 0" />
+            <origin xyz="9.97732e-19 -7.32058e-19 0.00731802" rpy="0 -0 0.742439" />
+            <inertia ixx="4.48843e-07" ixy="4.20673e-10" ixz="0" iyy="4.4877e-07" iyz="0" izz="5.69462e-07" />
+        </inertial>
+        <visual>
+            <origin xyz="0 0 0" rpy="0 -0 0.742439" />
             <geometry>
                 <mesh filename="package://drone_description/meshes/Motor_link.stl" scale="1 1 1" />
@@ -195,4 +261,10 @@
             </material>
         </visual>
+        <collision>
+            <origin xyz="0 0 0" rpy="0 -0 0.742439" />
+            <geometry>
+                <mesh filename="package://drone_description/meshes/Motor_link.stl" scale="1 1 1" />
+            </geometry>
+        </collision>
     </link>
     <link name="pillar_link">
@@ -211,4 +283,10 @@
             </material>
         </visual>
+        <collision>
+            <origin xyz="0 -7.65404e-20 -0.0039" rpy="0 -0 0" />
+            <geometry>
+                <mesh filename="package://drone_description/meshes/Pillar_link.stl" scale="1 1 1" />
+            </geometry>
+        </collision>
     </link>
     <link name="pillar_link_1">
@@ -227,4 +305,10 @@
             </material>
         </visual>
+        <collision>
+            <origin xyz="0 -7.65404e-20 -0.0039" rpy="0 -0 0" />
+            <geometry>
+                <mesh filename="package://drone_description/meshes/Pillar_link.stl" scale="1 1 1" />
+            </geometry>
+        </collision>
     </link>
     <link name="pillar_link_2">
@@ -243,4 +327,10 @@
             </material>
         </visual>
+        <collision>
+            <origin xyz="0 -7.65404e-20 -0.0039" rpy="0 -0 0" />
+            <geometry>
+                <mesh filename="package://drone_description/meshes/Pillar_link.stl" scale="1 1 1" />
+            </geometry>
+        </collision>
     </link>
     <link name="pillar_link_3">
@@ -259,4 +349,10 @@
             </material>
         </visual>
+        <collision>
+            <origin xyz="0 -7.65404e-20 -0.0039" rpy="0 -0 0" />
+            <geometry>
+                <mesh filename="package://drone_description/meshes/Pillar_link.stl" scale="1 1 1" />
+            </geometry>
+        </collision>
     </link>
     <link name="propeller_link">
@@ -339,4 +435,10 @@
             </material>
         </visual>
+        <collision>
+            <origin xyz="0 -9.18485e-20 0" rpy="0 -0 0" />
+            <geometry>
+                <mesh filename="package://drone_description/meshes/Spacer_link.stl" scale="1 1 1" />
+            </geometry>
+        </collision>
     </link>
     <link name="spacer_link_1">
@@ -355,4 +457,10 @@
             </material>
         </visual>
+        <collision>
+            <origin xyz="0 -9.18485e-20 0" rpy="0 -0 0" />
+            <geometry>
+                <mesh filename="package://drone_description/meshes/Spacer_link.stl" scale="1 1 1" />
+            </geometry>
+        </collision>
     </link>
     <link name="spacer_link_2">
@@ -371,4 +479,10 @@
             </material>
         </visual>
+        <collision>
+            <origin xyz="0 -9.18485e-20 0" rpy="0 -0 0" />
+            <geometry>
+                <mesh filename="package://drone_description/meshes/Spacer_link.stl" scale="1 1 1" />
+            </geometry>
+        </collision>
     </link>
     <link name="spacer_link_3">
@@ -387,4 +501,10 @@
             </material>
         </visual>
+        <collision>
+            <origin xyz="0 -9.18485e-20 0" rpy="0 -0 0" />
+            <geometry>
+                <mesh filename="package://drone_description/meshes/Spacer_link.stl" scale="1 1 1" />
+            </geometry>
+        </collision>
     </link>
     <link name="spinner_link">
@@ -455,9 +575,9 @@
         <inertial>
             <mass value="0.0175978" />
-            <origin xyz="3.72278e-18 -6.70824e-18 0.00162799" rpy="0 -0 0" />
+            <origin xyz="-0.0311127 0.0226274 -0.00247201" rpy="0 -0 0" />
             <inertia ixx="8.7077e-06" ixy="0" ixz="0" iyy="8.88847e-06" iyz="0" izz="1.75536e-05" />
         </inertial>
         <visual>
-            <origin xyz="0 0 0" rpy="0 -0 0" />
+            <origin xyz="-0.0311127 0.0226274 -0.0041" rpy="0 -0 0" />
             <geometry>
                 <mesh filename="package://drone_description/meshes/Top_link.stl" scale="1 1 1" />
@@ -467,31 +587,37 @@
             </material>
         </visual>
-    </link>
-    <joint name="arms_top_1_joint" type="fixed">
-        <origin xyz="0.0311127 -0.0226274 0.0041" rpy="-3.14159 -4.28599e-17 0.785398" />
+        <collision>
+            <origin xyz="-0.0311127 0.0226274 -0.0041" rpy="0 -0 0" />
+            <geometry>
+                <mesh filename="package://drone_description/meshes/Top_link.stl" scale="1 1 1" />
+            </geometry>
+        </collision>
+    </link>
+    <joint name="arm_top_1_joint" type="fixed">
+        <origin xyz="1.80411e-16 1.70003e-16 0.02" rpy="3.14159 7.61702e-16 1.5708" />
         <axis xyz="-0 -0 1" />
-        <parent link="top_link" />
-        <child link="arm_link" />
+        <parent link="arm_link" />
+        <child link="top_link" />
     </joint>
     <joint name="base_board1_joint" type="fixed">
-        <origin xyz="0.0463627 0.00737742 -0.0005" rpy="2.11916e-17 -4.90352e-18 -4.996e-16" />
+        <origin xyz="0.01525 -0.01525 0.0075" rpy="2.22283e-16 -3.92282e-17 -1.77636e-15" />
         <axis xyz="0 0 -1" />
         <parent link="base_link" />
         <child link="board_link" />
     </joint>
+    <joint name="base_joint" type="fixed">
+        <origin xyz="-1.56913e-19 8.43865e-19 -1.38778e-17" rpy="-3.82105e-31 6.02855e-61 3.15544e-30" />
+        <axis xyz="-0 -0 -1" />
+        <parent link="root" />
+        <child link="base_link" />
+    </joint>
     <joint name="board2_imu_joint" type="fixed">
-        <origin xyz="0.01525 0.01525 -0.00175" rpy="-3.14159 1.38667e-32 -3.14159" />
+        <origin xyz="0.01525 0.01525 -0.00175" rpy="-3.14159 1.2326e-32 3.14159" />
         <axis xyz="0 0 -1" />
         <parent link="board_link_1" />
         <child link="imu_link" />
     </joint>
-    <joint name="hanging_node_to_root_joint" type="fixed">
-        <origin xyz="-0.0814963 0.0335523 0.0258382" rpy="-3.14159 2.13437e-16 -2.39915" />
-        <axis xyz="0 0 1" />
-        <parent link="root" />
-        <child link="top_link" />
-    </joint>
     <joint name="motor1_spinner1_joint" type="continuous">
-        <origin xyz="2.77556e-17 1.38778e-17 0.0185" rpy="-7.64093e-18 3.26804e-18 0.0429589" />
+        <origin xyz="4.19227e-18 -2.77556e-17 0.0185" rpy="-1.47326e-16 6.30118e-17 0.785398" />
         <axis xyz="-0 -0 -1" />
         <parent link="motor_link_1" />
@@ -499,5 +625,5 @@
     </joint>
     <joint name="motor2_spinner2_joint" type="continuous">
-        <origin xyz="0 3.46945e-18 0.0185" rpy="-8.55285e-50 2.46519e-32 -6.93889e-18" />
+        <origin xyz="1.38778e-17 1.32506e-18 0.0185" rpy="2.29353e-32 -2.31216e-32 0.742439" />
         <axis xyz="0 0 -1" />
         <parent link="motor_link_3" />
@@ -505,5 +631,5 @@
     </joint>
     <joint name="motor3_spinner3_joint" type="continuous">
-        <origin xyz="0 2.77556e-17 0.0185" rpy="0 -0 2.902e-33" />
+        <origin xyz="-7.74265e-19 -1.38778e-17 0.0185" rpy="4.9128e-32 -3.33176e-32 0.742439" />
         <axis xyz="0 0 -1" />
         <parent link="motor_link" />
@@ -511,5 +637,5 @@
     </joint>
     <joint name="motor4_spinner4_joint" type="continuous">
-        <origin xyz="0 0 0.0185" rpy="1.2326e-32 1.2326e-32 -6.93889e-18" />
+        <origin xyz="1.38778e-17 -1.33374e-18 0.0185" rpy="2.84368e-32 4.57052e-32 0.742439" />
         <axis xyz="0 0 -1" />
         <parent link="motor_link_2" />
@@ -517,5 +643,5 @@
     </joint>
     <joint name="rear_left_arm_base_1_joint" type="fixed">
-        <origin xyz="0.00848528 0.0537401 -8.67362e-19" rpy="1.11911e-17 -1.72107e-17 1.94289e-16" />
+        <origin xyz="-0.0226274 0.0311127 0.008" rpy="-3.02751e-16 1.17373e-16 -1.33227e-15" />
         <axis xyz="0 0 -1" />
         <parent link="base_link" />
@@ -523,5 +649,5 @@
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